Commit message: Ridgeback for lasa

File: ridgeback_description/urdf/accessories.urdf.xacro (robot description, xacro)
@@ -11,4 +11,5 @@
   <xacro:include filename="$(find ridgeback_description)/urdf/accessories/sick_lms1xx_mount.urdf.xacro" />
   <xacro:include filename="$(find ridgeback_description)/urdf/accessories/hokuyo_ust-10lx_mount.urdf.xacro" />
+  <xacro:include filename="$(find ur_description)/urdf/ur5.urdf.xacro" />
   <!-- If enabled, generate the front HOKUYO UST-10LX LASER payload. -->
   <xacro:if value="$(optenv RIDGEBACK_FRONT_HOKUYO_LASER 0)">
@@ -35,3 +36,47 @@
                             location="-1" />
   </xacro:if>
+  <link name="arch_link">
+		<visual>
+			<geometry>
+				<mesh filename="package://ridgeback_description/meshes/epfl_arch.dae" />
+			</geometry>
+		</visual>
+		<collision>
+			<geometry>
+				<mesh filename="package://ridgeback_description/meshes/epfl_arch.dae" />
+			</geometry>
+		</collision>
+   </link>
+  <joint name="arch_joint" type="fixed">
+	  <origin xyz="-0.38 0 0.278" rpy="0 0 1.5" />
+	  <parent link="top_link" />
+	  <child link="arch_link" />
+  </joint>
+<!-- Spawn arm -->
+  <xacro:ur5_robot prefix="ur5_arm_" joint_limited="true"/>
+  <!-- Join arm -->
+  <joint name="ur5_arm_base" type="fixed">
+	<parent link="mid_mount" />
+	<child link="ur5_arm_base_link" />
+	<origin xyz="0.22 0.0 0.0" rpy="0.0 0.0 -1.5708" />
+  </joint>
+  <!-- Sensor Mount and other custom parts -->
+  <link name="FT300_link">
+		<visual>
+			<geometry>
+				<cylinder length="0.04" radius="0.035"/>
+			</geometry>
+			<material name="black"/>
+		</visual>
+		<collision>
+			<geometry>
+				<cylinder length="0.04" radius="0.035"/>
+			</geometry>
+		</collision>
+   </link>
+  <joint name="FT300_joint" type="fixed">
+	  <origin xyz="0.02 0 0" rpy="0 1.57 0" />
+	  <parent link="ur5_arm_ee_link" />
+	  <child link="FT300_link" />
+  </joint>
 </robot>

File: ridgeback_description/urdf/ridgeback.urdf.xacro (robot description, xacro)
@@ -11,7 +11,4 @@
   <xacro:property name="rocker_offset" value="0.319" />
   <xacro:property name="rocker_width" value="0.472" />
-  <xacro:property name="imu_offset_x" value="0.2085" />
-  <xacro:property name="imu_offset_y" value="-0.2902" />
-  <xacro:property name="imu_offset_z" value="0.1681" />
   <xacro:property name="dummy_inertia" value="1e-09"/>
   <material name="dark_grey"><color rgba="0.2 0.2 0.2 1.0" /></material>
@@ -19,4 +16,5 @@
   <material name="yellow"><color rgba="0.8 0.8 0.0 1.0" /></material>
   <material name="black"><color rgba="0.15 0.15 0.15 1.0" /></material>
+  <xacro:include filename="$(find ur_description)/urdf/ur5.urdf.xacro" />
   <xacro:macro name="wheel" params="prefix side *joint_pose">
     <link name="${prefix}_${side}_wheel_link">
@@ -192,5 +190,4 @@
     <parent link="chassis_link" />
     <child link="imu_link" />
-    <origin xyz="${imu_offset_x} ${imu_offset_y} ${imu_offset_z}" rpy="0 0 0"/>
   </joint>
   <link name="mid_mount" />
